Commit message: fixed unable to load meshes as visual elements

File: maskor_ev3/description/urdf/bobb3e/mindstorm_second.urdf (robot description, URDF)
Before this commit: robot mindstorm, 11 links, 10 joints
Links:
- link base_link: geometry collision box size=1 0.6 0.2; visual mesh filename=package://maskor_ev3/description/meshes/bobb3e_baseLink.dae scale=1 1 1

Commit message: mindstorm_second modified

File: maskor_ev3/description/urdf/bobb3e/mindstorm_second.urdf (robot description, URDF)
Before this commit: robot mindstorm, 11 links, 10 joints
Links:
- link color_sensor_box: geometry collision box size=0.15 0.05 0.05
- link ir_sensor_box: geometry collision box size=0.05 0.2 0.05
- link left_fork: geometry collision box size=0.5 0.05 0.05
- link lift_left: geometry collision box size=0.1 0.05 1
- link lift_right: geometry collision box size=0.1 0.05 1
- link lift_top: geometry collision box size=0.1 0.45 0.05
- link right_fork: geometry collision box size=0.5 0.05 0.05
- link slider: geometry collision box size=0.05 0.5 0.045

Commit message: urdf fixes and launch fixes

File: maskor_ev3/description/urdf/bobb3e/mindstorm_second.urdf (robot description, URDF)
Before this commit: robot mindstorm, 11 links, 10 joints
Links:
- removed link caster_wheel
- removed link color_sensor_box
- removed link gegengewicht
- removed link ir_sensor_box
- removed link left_fork
- removed link lift_left
- removed link lift_right
- removed link lift_top
- removed link right_fork
- removed link slider
- added link base_foot_print; collision box size=0.1 0.06 0.02; visual box size=0.1 0.06 0.02
- added link left_wheel; visual cylinder length=0.075 radius=0.08
- link base_link: geometry collision box size=0.005 0.005 0.005; visual box size=0.005 0.005 0.005
Joints:
- removed joint caster_wheel_joint
- removed joint color_sensor_box_joint
- removed joint fork_left_joint
- removed joint fork_right_joint
- removed joint gegengewicht_joint
- removed joint ir_sensor_box_joint
- removed joint lift_joint_left
- removed joint lift_joint_right
- removed joint lift_joint_top
- removed joint slider_joint
- added joint base_link_joint: type fixed, parent base_foot_print, child base_link, origin xyz=0 0 0.002
- added joint head_swivel: type continuous, parent base_link, child left_wheel, origin xyz=0 0 0.3, axis 0 0 1

Commit message: changes in urdf and launch

File: maskor_ev3/description/urdf/bobb3e/mindstorm_second.urdf (robot description, URDF)
Before this commit: robot mindstorm, 3 links, 2 joints
Links:
- removed link base_foot_print
- removed link left_wheel
- added link caster_wheel; collision sphere radius=0.05; visual sphere radius=0.05
- added link color_sensor_box; collision box size=0.15 0.05 0.05
- added link gegengewicht; collision box size=0.05 0.05 0.05; visual box size=0.05 0.05 0.05
- added link ir_sensor_box; collision box size=0.05 0.2 0.05
- added link left_fork; collision box size=0.5 0.05 0.05
- added link lift_left; collision box size=0.1 0.05 1
- added link lift_right; collision box size=0.1 0.05 1
- added link lift_top; collision box size=0.1 0.45 0.05
- added link right_fork; collision box size=0.5 0.05 0.05
- added link slider; collision box size=0.05 0.5 0.045
- link base_link: geometry collision box size=1 0.6 0.2; visual mesh filename=package://maskor_ev3/description/meshes/bobb3e_baseLink.dae scale=1 1 1
Joints:
- removed joint base_link_joint
- removed joint head_swivel
- added joint caster_wheel_joint: type continuous, parent base_link, child caster_wheel, origin xyz=-0.3 0 -0.155, axis 0 1 0
- added joint color_sensor_box_joint: type fixed, parent base_link, child color_sensor_box, origin xyz=0.5 0 -0.1 rpy=0 1.5708 0
- added joint fork_left_joint: type fixed, parent slider, child left_fork, origin xyz=0 0 0
- added joint fork_right_joint: type fixed, parent slider, child right_fork, origin xyz=0 0 0
- added joint gegengewicht_joint: type fixed, parent base_link, child gegengewicht, origin xyz=-0.3 0 0
- added joint ir_sensor_box_joint: type fixed, parent base_link, child ir_sensor_box, origin xyz=0.5 0 0.05
- added joint lift_joint_left: type fixed, parent base_link, child lift_left, origin xyz=0.55 0 0.35
- added joint lift_joint_right: type fixed, parent base_link, child lift_right, origin xyz=0.55 0 0.35
- added joint lift_joint_top: type fixed, parent base_link, child lift_top, origin xyz=0.55 0 0.35
- added joint slider_joint: type prismatic, parent lift_left, child slider, origin xyz=0.05 0 -0.5, axis 0 0 1, limit lower=0.0 upper=0.8 effort=1000.0 velocity=0.5
