Commit message: added 2 more wheels to fake the tracks and added joint_state_publisher to launch file

File: maskor_ev3/description/urdf/bobb3e/maskor_ev3_bobb3e.urdf (robot description, URDF)
Before this commit: robot maskor_ev3_bobb3e, 7 links, 6 joints
Links:
- removed link left_wheel_link
- removed link right_wheel_link
- added link left_front_wheel_link; collision cylinder length=0.08 radius=0.075; visual mesh filename=package://maskor_ev3/description/meshes/bobb3e_tire.dae scale=1 1 1
- added link left_rear_wheel_link; collision cylinder length=0.08 radius=0.075; visual mesh filename=package://maskor_ev3/description/meshes/bobb3e_tire.dae scale=1 1 1
- added link right_front_wheel_link; collision cylinder length=0.08 radius=0.075; visual mesh filename=package://maskor_ev3/description/meshes/bobb3e_tire.dae scale=1 1 1
- added link right_rear_wheel_link; collision cylinder length=0.08 radius=0.075; visual mesh filename=package://maskor_ev3/description/meshes/bobb3e_tire.dae scale=1 1 1
- link base_link: mass None -> 0.1
- link fork_lift_link: mass None -> 0.1
Joints:
- removed joint base_link_to_left_wheel
- removed joint base_link_to_right_wheel
- added joint base_link_to_left_front_wheel: type continuous, parent base_link, child left_front_wheel_link, origin xyz=0.03 0.03 0, axis 0 1 0
- added joint base_link_to_left_rear_wheel: type continuous, parent base_link, child left_rear_wheel_link, origin xyz=-0.03 0.03 0, axis 0 1 0
- added joint base_link_to_right_front_wheel: type continuous, parent base_link, child right_front_wheel_link, origin xyz=0.03 -0.03 0, axis 0 1 0
- added joint base_link_to_right_rear_wheel: type continuous, parent base_link, child right_rear_wheel_link, origin xyz=-0.03 -0.03 0, axis 0 1 0
- joint base_link_to_fork_lift: axis (none) -> 0 0 1; limit (none) -> lower=-0.38 upper=0 effort=1000.0 velocity=0.5; origin xyz=0.05 -0.00 0.05 -> xyz=0.05 -0.00 1.05 rpy=0 0 0; type fixed -> prismatic

Commit message: added fake forklift joint

File: maskor_ev3/description/urdf/bobb3e/maskor_ev3_bobb3e.urdf (robot description, URDF)
Before this commit: robot maskor_ev3_bobb3e, 9 links, 8 joints
Links:
- added link infrared_sensor_link; collision box size=0.01 0.01 0.01; visual box size=0.01 0.01 0.01
- link base_footprint: geometry 
- link base_link: geometry collision box size=0.005 0.005 0.005; visual mesh filename=package://maskor_ev3/description/meshes/bobb3e_baseLink.dae scale=1 1 1
Joints:
- added joint base_link_to_infrared_sensor: type fixed, parent base_link, child infrared_sensor_link, origin xyz=0 0 0.12
- joint base_link_to_color_sensor: origin xyz=0.05 -0.00 0.005 -> xyz=0.1 -0.00 -0.035 rpy=0 1.5708 0
- joint base_link_to_fork_lift: limit lower=-0.38 upper=0 effort=1000.0 velocity=0.5 -> lower=0 upper=0.15 effort=1000.0 velocity=0.5; origin xyz=0.05 -0.00 1.05 rpy=0 0 0 -> xyz=0.1 -0.00 -0.05 rpy=0 0 0
- joint base_link_to_gyro_sensor: origin xyz=-0.03 -0.01 0.1 -> xyz=-0.03 -0.06 0.075
- joint base_link_to_left_front_wheel: origin xyz=0.03 0.03 0 -> xyz=0.03 0.065 -0.05
- joint base_link_to_left_rear_wheel: origin xyz=-0.03 0.03 0 -> xyz=-0.03 0.065 -0.05
- joint base_link_to_right_front_wheel: origin xyz=0.03 -0.03 0 -> xyz=0.03 -0.065 -0.05
- joint base_link_to_right_rear_wheel: origin xyz=-0.03 -0.03 0 -> xyz=-0.03 -0.065 -0.05

Commit message: added fork (a bad one)

File: maskor_ev3/description/urdf/bobb3e/maskor_ev3_bobb3e.urdf (robot description, URDF)
Before this commit: robot maskor_ev3_bobb3e, 10 links, 9 joints
Links:
- added link fork_link; collision box size=0.01 0.1 0.01; visual box size=0.01 0.1 0.01
- added link left_fork_link; collision box size=0.1 0.01 0.01; visual box size=0.1 0.01 0.01
- added link right_fork_link; collision box size=0.1 0.01 0.01; visual box size=0.1 0.01 0.01
- link fork_lift_link: geometry collision box size=0.01 0.01 0.01; visual box size=0.01 0.01 0.035
Joints:
- added joint fork_lift_link_to_fork_link: type fixed, parent fork_lift_link, child fork_link, origin xyz=0 0 0
- added joint fork_link_to_left_fork: type fixed, parent fork_link, child left_fork_link, origin xyz=0 -0.05 0
- added joint fork_link_to_right_fork: type fixed, parent fork_link, child right_fork_link, origin xyz=0 0.05 0
- joint base_link_to_fork_lift: origin xyz=0.1 -0.00 -0.05 rpy=0 0 0 -> xyz=0.1 -0.00 -0.035 rpy=0 0 0

Commit message: change urdf and add meshes

File: maskor_ev3/description/urdf/bobb3e/maskor_ev3_bobb3e.urdf (robot description, URDF)
Before this commit: robot maskor_ev3_bobb3e, 13 links, 12 joints
Links:
- link base_link: geometry collision box size=0.0198 0.017 0.0198; visual mesh filename=package://maskor_ev3/description/meshes/bobb3e_baseLink.dae scale=1 1 1
- link color_sensor_link: geometry collision box size=0.002 0.002 0.004; visual box size=0.01 0.01 0.035
- link gyro_sensor_link: geometry collision box size=0.002 0.002 0.004; visual box size=0.01 0.01 0.01
- link infrared_sensor_link: geometry collision box size=0.0045 0.0055 0.0023; visual box size=0.0045 0.0055 0.0023
- link left_front_wheel_link: mass None -> 0.1; geometry collision cylinder length=0.02 radius=0.015; visual mesh filename=package://maskor_ev3/description/meshes/bobb3e_tire.dae scale=1 1 1
- link left_rear_wheel_link: mass None -> 0.1; geometry collision cylinder length=0.02 radius=0.015; visual mesh filename=package://maskor_ev3/description/meshes/bobb3e_tire.dae scale=1 1 1
- link right_front_wheel_link: mass None -> 0.1; geometry collision cylinder length=0.02 radius=0.015; visual mesh filename=package://maskor_ev3/description/meshes/bobb3e_tire.dae scale=1 1 1
- link right_rear_wheel_link: mass None -> 0.1; geometry collision cylinder length=0.02 radius=0.015; visual mesh filename=package://maskor_ev3/description/meshes/bobb3e_tire.dae scale=1 1 1
Joints:
- joint base_link_to_base_footprint: origin xyz=0 0 0.05 -> xyz=0 0 0
- joint base_link_to_left_front_wheel: origin xyz=0.03 0.065 -0.05 -> xyz=0.0475 0.065 0.022
- joint base_link_to_left_rear_wheel: origin xyz=-0.03 0.065 -0.05 -> xyz=-0.0475 0.065 0.022
- joint base_link_to_right_front_wheel: origin xyz=0.03 -0.065 -0.05 -> xyz=0.0475 -0.065 0.022
- joint base_link_to_right_rear_wheel: origin xyz=-0.03 -0.065 -0.05 -> xyz=-0.0475 -0.065 0.022

Commit message: modified meshes and urdf

File: maskor_ev3/description/urdf/bobb3e/maskor_ev3_bobb3e.urdf (robot description, URDF)
Before this commit: robot maskor_ev3_bobb3e, 13 links, 12 joints
Links:
- link fork_lift_link: geometry collision box size=0.01 0.089 0.064; visual mesh filename=package://maskor_ev3/description/meshes/bobb3e_fork_lift.dae scale=1 1 1
Joints:
- removed joint base_link_to_fork_lift
- added joint base_link_to_fork_lift_link: type prismatic, parent base_link, child fork_lift_link, origin xyz=0.1 0 0.02 rpy=0 0 0, axis 0 0 1, limit lower=0 upper=0.15 effort=1000.0 velocity=0.5
- joint base_link_to_color_sensor: origin xyz=0.1 -0.00 -0.035 rpy=0 1.5708 0 -> xyz=0.1 -0.00 0.02 rpy=0 1.5708 0
- joint base_link_to_infrared_sensor: origin xyz=0 0 0.12 -> xyz=0 0 0.18
- joint fork_link_to_left_fork: origin xyz=0 -0.05 0 -> xyz=0 0.015 0
- joint fork_link_to_right_fork: origin xyz=0 0.05 0 -> xyz=0 -0.015 0

Commit message: fixed mesh and mod. urdf

File: maskor_ev3/description/urdf/bobb3e/maskor_ev3_bobb3e.urdf (robot description, URDF)
Before this commit: robot maskor_ev3_bobb3e, 13 links, 12 joints
Links:
- removed link fork_link
- added link left_fork_arm_link; visual mesh filename=package://maskor_ev3/description/meshes/bobb3e_arm_left.dae scale=1 1 1
- link left_fork_link: geometry collision box size=0.073 0.016 0.01
- link right_fork_link: geometry collision box size=0.073 0.016 0.01
Joints:
- removed joint fork_lift_link_to_fork_link
- added joint base_link_to_left_fork_arm: type continuous, parent base_link, child left_fork_arm_link, origin xyz=-0.024 0.05 0.1125 rpy=0 0 3.14159, axis 0 1 0
- joint base_link_to_fork_lift_link: limit lower=0 upper=0.15 effort=1000.0 velocity=0.5 -> lower=0.01 upper=0.15 effort=50.0 velocity=0.5; origin xyz=0.1 0 0.02 rpy=0 0 0 -> xyz=0.11 0 0.02 rpy=0 0 0
- joint fork_link_to_left_fork: parent fork_link -> fork_lift_link
- joint fork_link_to_right_fork: parent fork_link -> fork_lift_link
