Commit message: modified URDF model to include package maskor_ev3_descrption as a source

File: maskor_ev3_description/urdf/bobb3e/maskor_ev3_bobb3e.urdf (robot description, URDF)
Before this commit: robot maskor_ev3_bobb3e, 13 links, 12 joints
Links:
- link base_link: geometry collision box size=0.0198 0.017 0.0198; visual mesh filename=package://maskor_ev3_description/meshes/bobb3e_baseLink.dae scale=1 1 1
- link fork_lift_link: geometry collision box size=0.01 0.089 0.064; visual mesh filename=package://maskor_ev3_description/meshes/bobb3e_fork_lift.dae scale=1 1 1
- link left_fork_arm_link: geometry visual mesh filename=package://maskor_ev3_description/meshes/bobb3e_arm_left.dae scale=1 1 1
- link left_front_wheel_link: geometry collision cylinder length=0.02 radius=0.015; visual mesh filename=package://maskor_ev3_description/meshes/bobb3e_tire.dae scale=1 1 1
- link left_rear_wheel_link: geometry collision cylinder length=0.02 radius=0.015; visual mesh filename=package://maskor_ev3_description/meshes/bobb3e_tire.dae scale=1 1 1
- link right_front_wheel_link: geometry collision cylinder length=0.02 radius=0.015; visual mesh filename=package://maskor_ev3_description/meshes/bobb3e_tire.dae scale=1 1 1
- link right_rear_wheel_link: geometry collision cylinder length=0.02 radius=0.015; visual mesh filename=package://maskor_ev3_description/meshes/bobb3e_tire.dae scale=1 1 1

Commit message: added fake visuals for forks to be able to apply material color for collision visualization

File: maskor_ev3_description/urdf/bobb3e/maskor_ev3_bobb3e.urdf (robot description, URDF)
Before this commit: robot maskor_ev3_bobb3e, 13 links, 12 joints
Links:
- link left_fork_link: geometry collision box size=0.073 0.016 0.01; visual box size=0.01 0.01 0.01
- link right_fork_link: geometry collision box size=0.073 0.016 0.01; visual box size=0.01 0.01 0.01

Commit message: re-positioned base_link

File: maskor_ev3_description/urdf/bobb3e/maskor_ev3_bobb3e.urdf (robot description, URDF)
Before this commit: robot maskor_ev3_bobb3e, 13 links, 12 joints
Links:
- link base_link: geometry collision box size=0.20 0.12 0.10; visual mesh filename=package://maskor_ev3_description/meshes/bobb3e_baseLink.dae scale=1 1 1
Joints:
- joint base_link_to_base_footprint: origin xyz=0 0 0 -> xyz=0 0 0.04
- joint base_link_to_left_front_wheel: origin xyz=0.0475 0.065 0.022 -> xyz=0.078 0.065 -0.018
- joint base_link_to_left_rear_wheel: origin xyz=-0.0475 0.065 0.022 -> xyz=-0.0175 0.065 -0.018
- joint base_link_to_right_front_wheel: origin xyz=0.0475 -0.065 0.022 -> xyz=0.078 -0.065 -0.018
- joint base_link_to_right_rear_wheel: origin xyz=-0.0475 -0.065 0.022 -> xyz=-0.0175 -0.065 -0.018

Commit message: re-positioned base_link

File: maskor_ev3_description/urdf/bobb3e/maskor_ev3_bobb3e.urdf (robot description, URDF)
Before this commit: robot maskor_ev3_bobb3e, 13 links, 12 joints
Joints:
- joint base_link_to_base_footprint: origin xyz=0 0 0.04 -> xyz=0 0 0.03

Commit message: re-positioned infrared_sensor_link

File: maskor_ev3_description/urdf/bobb3e/maskor_ev3_bobb3e.urdf (robot description, URDF)
Before this commit: robot maskor_ev3_bobb3e, 13 links, 12 joints
Joints:
- joint base_link_to_infrared_sensor: origin xyz=0 0 0.18 -> xyz=0 0 0.15

Commit message: added some basic collision boxed for all needed components

File: maskor_ev3_description/urdf/bobb3e/maskor_ev3_bobb3e.urdf (robot description, URDF)
Before this commit: robot maskor_ev3_bobb3e, 13 links, 12 joints
Links:
- link base_link: geometry collision box size=0.165 0.105 0.12; visual mesh filename=package://maskor_ev3_description/meshes/bobb3e_baseLink.dae scale=1 1 1
- link color_sensor_link: geometry collision box size=0.025 0.025 0.045; visual box size=0.001 0.001 0.001
- link infrared_sensor_link: geometry collision box size=0.055 0.065 0.03; visual box size=0.01 0.01 0.01
Joints:
- joint base_link_to_color_sensor: origin xyz=0.1 -0.00 0.02 rpy=0 1.5708 0 -> xyz=0.1 -0.00 -0.02 rpy=0 1.5708 0

Commit message: added fake left fork lift arm

File: maskor_ev3_description/urdf/bobb3e/maskor_ev3_bobb3e.urdf (robot description, URDF)
Before this commit: robot maskor_ev3_bobb3e, 13 links, 12 joints
Joints:
- joint base_link_to_fork_lift_link: limit lower=0.01 upper=0.15 effort=50.0 velocity=0.5 -> lower=-0.025 upper=0.11 effort=50.0 velocity=0.5
- joint base_link_to_left_fork_arm: limit (none) -> lower=-0.50 upper=0.50 effort=50.0 velocity=0.5; origin xyz=-0.024 0.05 0.1125 rpy=0 0 3.14159 -> xyz=-0.01 0.05 0.07 rpy=0 0 0; type continuous -> revolute

Commit message: added right fake arm for the fork lift

File: maskor_ev3_description/urdf/bobb3e/maskor_ev3_bobb3e.urdf (robot description, URDF)
Before this commit: robot maskor_ev3_bobb3e, 13 links, 12 joints
Links:
- added link right_fork_arm_link; visual mesh filename=package://maskor_ev3_description/meshes/bobb3e_arm_left.dae scale=1 1 1
Joints:
- added joint base_link_to_right_fork_arm: type revolute, parent base_link, child right_fork_arm_link, origin xyz=-0.01 -0.05 0.07 rpy=0 0 0, axis 0 1 0, limit lower=-0.50 upper=0.50 effort=50.0 velocity=0.5

Commit message: increased  mass of base link => removes jittering

File: maskor_ev3_description/urdf/bobb3e/maskor_ev3_bobb3e.urdf (robot description, URDF)
Before this commit: robot maskor_ev3_bobb3e, 14 links, 13 joints
Links:
- link base_link: mass 0.1 -> 5.0; geometry collision box size=0.165 0.105 0.20; visual mesh filename=package://maskor_ev3_description/meshes/bobb3e_baseLink.dae scale=1 1 1

Commit message: increased weight ratio between base link and wheels

File: maskor_ev3_description/urdf/bobb3e/maskor_ev3_bobb3e.urdf (robot description, URDF)
Before this commit: robot maskor_ev3_bobb3e, 14 links, 13 joints
Links:
- link base_link: mass 5.0 -> 20.0; geometry collision box size=0.165 0.105 0.12; visual mesh filename=package://maskor_ev3_description/meshes/bobb3e_baseLink.dae scale=1 1 1
- link left_front_wheel_link: mass 0.1 -> ${wheel_mass}
- link left_rear_wheel_link: mass 0.1 -> ${wheel_mass}
- link right_front_wheel_link: mass 0.1 -> ${wheel_mass}
- link right_rear_wheel_link: mass 0.1 -> ${wheel_mass}

Commit message: added friction to wheel joints

File: maskor_ev3_description/urdf/bobb3e/maskor_ev3_bobb3e.urdf (robot description, URDF)
Before this commit: robot maskor_ev3_bobb3e, 14 links, 13 joints
Links:
- link base_link: mass 20.0 -> 5.0

Commit message: change base link collision

File: maskor_ev3_description/urdf/bobb3e/maskor_ev3_bobb3e.urdf (robot description, URDF)
Before this commit: robot maskor_ev3_bobb3e, 14 links, 13 joints
Links:
- link base_link: mass 5.0 -> 1.0; geometry collision box size=0.125 0.105 0.07; visual mesh filename=package://maskor_ev3_description/meshes/bobb3e_baseLink.dae scale=1 1 1

Commit message: add fork_torque

File: maskor_ev3_description/urdf/bobb3e/maskor_ev3_bobb3e.urdf (robot description, URDF)
Before this commit: robot maskor_ev3_bobb3e, 14 links, 13 joints
Links:
- link base_link: mass 1.0 -> 5.0

Commit message: smal urdf modification

File: maskor_ev3_description/urdf/bobb3e/maskor_ev3_bobb3e.urdf (robot description, URDF)
Before this commit: robot maskor_ev3_bobb3e, 14 links, 13 joints
Links:
- link base_link: mass 5.0 -> 1.0

Commit message: update urdf

File: maskor_ev3_description/urdf/bobb3e/maskor_ev3_bobb3e.urdf (robot description, URDF)
Before this commit: robot maskor_ev3_bobb3e, 14 links, 13 joints
Links:
- link left_fork_link: mass 0.1 -> None
- link right_fork_link: mass 0.1 -> None

Commit message: create test.launch and test plugin in kinetic

File: maskor_ev3_description/urdf/bobb3e/maskor_ev3_bobb3e.urdf (robot description, URDF)
Before this commit: robot maskor_ev3_bobb3e, 14 links, 13 joints
Links:
- link left_front_wheel_link: mass ${wheel_mass} -> 3.0
- link left_rear_wheel_link: mass ${wheel_mass} -> 3.0
- link right_front_wheel_link: mass ${wheel_mass} -> 3.0
- link right_rear_wheel_link: mass ${wheel_mass} -> 3.0

Commit message: add camera plugin

File: maskor_ev3_description/urdf/bobb3e/maskor_ev3_bobb3e.urdf (robot description, URDF)
Before this commit: robot maskor_ev3_bobb3e, 14 links, 13 joints
Joints:
- joint base_link_to_color_sensor: origin xyz=0.1 -0.00 -0.02 rpy=0 1.5708 0 -> xyz=0.1 -0.0 -0.01 rpy=0 1.5708 0

Commit message: add infrared sensor

File: maskor_ev3_description/urdf/bobb3e/maskor_ev3_bobb3e.urdf (robot description, URDF)
Before this commit: robot maskor_ev3_bobb3e, 14 links, 13 joints
Joints:
- joint base_link_to_infrared_sensor: origin xyz=0 0 0.15 -> xyz=0 0 0.15 rpy=0 0.5 0

Commit message: added first working version of the gyro sensor plugin (needs to be veryfied against the real sensor)

File: maskor_ev3_description/urdf/bobb3e/maskor_ev3_bobb3e.urdf (robot description, URDF)
Before this commit: robot maskor_ev3_bobb3e, 14 links, 13 joints
Links:
- link gyro_sensor_link: geometry collision box size=0.002 0.002 0.004; visual box size=0.002 0.002 0.004
